Commit message: Fix origin/rotation of most STLs

File: ros/wall_e_description/urdf/wall_e.urdf.xacro (robot description, xacro)
@@ -15,9 +15,9 @@
     <parent link="base_footprint"/>
     <child link="base_link"/>
-    <origin xyz="0.0 0.0 0.15" rpy="0.0 0.0 0.0"/> <!--TODO fix offset of link-->
+    <origin xyz="0.0 0.0 0.138887" rpy="0.0 0.0 0.0"/> <!--TODO fix offset of link-->
   </joint>
   <link name="base_link">
     <visual>
-      <origin xyz="0.15 -0.15 -0.15" rpy="0.0 0.0 1.570796327"/> <!--TODO fix origin of mesh-->
+      <origin xyz="0.0 0.0 0.0" rpy="0.0 0.0 0.0"/>
       <geometry>
         <mesh filename="package://wall_e_description/meshes/body.stl" scale="0.001 0.001 0.001"/>
@@ -33,5 +33,5 @@
   <link name="drivetrain_right_link">
     <visual>
-      <origin xyz="0.15 -0.15 -0.15" rpy="0.0 0.0 1.570796327"/> <!--TODO fix origin of mesh-->
+      <origin xyz="0.0 0.0 0.0" rpy="0.0 0.0 0.0"/>
       <geometry>
         <mesh filename="package://wall_e_description/meshes/drivetrain-right.stl" scale="0.001 0.001 0.001"/>
@@ -47,5 +47,5 @@
   <link name="drivetrain_left_link">
     <visual>
-      <origin xyz="0.15 -0.15 -0.15" rpy="0.0 0.0 1.570796327"/> <!--TODO fix origin of mesh-->
+      <origin xyz="0.0 0.0 0.0" rpy="0.0 0.0 0.0"/>
       <geometry>
         <mesh filename="package://wall_e_description/meshes/drivetrain-left.stl" scale="0.001 0.001 0.001"/>
@@ -54,28 +54,28 @@
     </visual>
   </link>
-  <joint name="track_right_joint" type="fixed">
+  <joint name="tread_right_joint" type="fixed">
     <parent link="drivetrain_right_link"/>
-    <child link="track_right_link"/>
-    <origin xyz="0.0 0.0 0.0" rpy="0.0 0.0 0.0"/>
-  </joint>
-  <link name="track_right_link">
-    <visual>
-      <origin xyz="0.15 -0.15 -0.15" rpy="0.0 0.0 1.570796327"/> <!--TODO fix origin of mesh-->
-      <geometry>
-        <mesh filename="package://wall_e_description/meshes/track-right.stl" scale="0.001 0.001 0.001"/>
+    <child link="tread_right_link"/>
+    <origin xyz="0.0 0.0 0.0" rpy="0.0 0.0 0.0"/>
+  </joint>
+  <link name="tread_right_link">
+    <visual>
+      <origin xyz="0.0 0.0 0.0" rpy="0.0 0.0 0.0"/>
+      <geometry>
+        <mesh filename="package://wall_e_description/meshes/tread-right.stl" scale="0.001 0.001 0.001"/>
       </geometry>
       <material name="black"/>
     </visual>
   </link>
-  <joint name="track_left_joint" type="fixed">
+  <joint name="tread_left_joint" type="fixed">
     <parent link="drivetrain_left_link"/>
-    <child link="track_left_link"/>
-    <origin xyz="0.0 0.0 0.0" rpy="0.0 0.0 0.0"/>
-  </joint>
-  <link name="track_left_link">
-    <visual>
-      <origin xyz="0.15 -0.15 -0.15" rpy="0.0 0.0 1.570796327"/> <!--TODO fix origin of mesh-->
-      <geometry>
-        <mesh filename="package://wall_e_description/meshes/track-left.stl" scale="0.001 0.001 0.001"/>
+    <child link="tread_left_link"/>
+    <origin xyz="0.0 0.0 0.0" rpy="0.0 0.0 0.0"/>
+  </joint>
+  <link name="tread_left_link">
+    <visual>
+      <origin xyz="0.0 0.0 0.0" rpy="0.0 0.0 0.0"/>
+      <geometry>
+        <mesh filename="package://wall_e_description/meshes/tread-left.stl" scale="0.001 0.001 0.001"/>
       </geometry>
       <material name="black"/>
@@ -89,5 +89,5 @@
   <link name="wheel_right_link">
     <visual>
-      <origin xyz="0.15 -0.15 -0.15" rpy="0.0 0.0 1.570796327"/> <!--TODO fix origin of mesh-->
+      <origin xyz="0.0 0.0 0.0" rpy="0.0 0.0 0.0"/> <!--TODO fix origin of mesh-->
       <geometry>
         <mesh filename="package://wall_e_description/meshes/wheel-right.stl" scale="0.001 0.001 0.001"/>
@@ -103,5 +103,5 @@
   <link name="wheel_left_link">
     <visual>
-      <origin xyz="0.15 -0.15 -0.15" rpy="0.0 0.0 1.570796327"/> <!--TODO fix origin of mesh-->
+      <origin xyz="0.0 0.0 0.0" rpy="0.0 0.0 0.0"/> <!--TODO fix origin of mesh-->
       <geometry>
         <mesh filename="package://wall_e_description/meshes/wheel-left.stl" scale="0.001 0.001 0.001"/>
@@ -117,5 +117,5 @@
   <link name="arm_right_link">
     <visual>
-      <origin xyz="0.15 -0.15 -0.15" rpy="0.0 0.0 1.570796327"/> <!--TODO fix origin of mesh-->
+      <origin xyz="0.0 0.0 0.0" rpy="0.0 0.0 0.0"/> <!--TODO fix origin of mesh-->
       <geometry>
         <mesh filename="package://wall_e_description/meshes/arm-right.stl" scale="0.001 0.001 0.001"/>
@@ -131,5 +131,5 @@
   <link name="arm_left_link">
     <visual>
-      <origin xyz="0.15 -0.15 -0.15" rpy="0.0 0.0 1.570796327"/> <!--TODO fix origin of mesh-->
+      <origin xyz="0.0 0.0 0.0" rpy="0.0 0.0 0.0"/> <!--TODO fix origin of mesh-->
       <geometry>
         <mesh filename="package://wall_e_description/meshes/arm-left.stl" scale="0.001 0.001 0.001"/>
@@ -145,5 +145,5 @@
   <link name="hand_right_link">
     <visual>
-      <origin xyz="0.15 -0.15 -0.15" rpy="0.0 0.0 1.570796327"/> <!--TODO fix origin of mesh-->
+      <origin xyz="0.0 0.0 0.0" rpy="0.0 0.0 0.0"/> <!--TODO fix origin of mesh-->
       <geometry>
         <mesh filename="package://wall_e_description/meshes/hand-right.stl" scale="0.001 0.001 0.001"/>
@@ -159,5 +159,5 @@
   <link name="hand_left_link">
     <visual>
-      <origin xyz="0.15 -0.15 -0.15" rpy="0.0 0.0 1.570796327"/> <!--TODO fix origin of mesh-->
+      <origin xyz="0.0 0.0 0.0" rpy="0.0 0.0 0.0"/> <!--TODO fix origin of mesh-->
       <geometry>
         <mesh filename="package://wall_e_description/meshes/hand-left.stl" scale="0.001 0.001 0.001"/>
@@ -173,5 +173,5 @@
   <link name="neck_bottom_link">
     <visual>
-      <origin xyz="0.15 -0.15 -0.15" rpy="0.0 0.0 1.570796327"/> <!--TODO fix origin of mesh-->
+      <origin xyz="0.0 0.0 0.0" rpy="0.0 0.0 0.0"/> <!--TODO fix origin of mesh-->
       <geometry>
         <mesh filename="package://wall_e_description/meshes/neck-bottom.stl" scale="0.001 0.001 0.001"/>
@@ -187,5 +187,5 @@
   <link name="neck_top_link">
     <visual>
-      <origin xyz="0.15 -0.15 -0.15" rpy="0.0 0.0 1.570796327"/> <!--TODO fix origin of mesh-->
+      <origin xyz="0. 0.0 0.0" rpy="0.0 0.0 0.0"/> <!--TODO fix origin of mesh-->
       <geometry>
         <mesh filename="package://wall_e_description/meshes/neck-top.stl" scale="0.001 0.001 0.001"/>
@@ -201,5 +201,5 @@
   <link name="head_center_link">
     <visual>
-      <origin xyz="0.15 -0.15 -0.15" rpy="0.0 0.0 1.570796327"/> <!--TODO fix origin of mesh-->
+      <origin xyz="0.0 0.0 0.0" rpy="0.0 0.0 0.0"/> <!--TODO fix origin of mesh-->
       <geometry>
         <mesh filename="package://wall_e_description/meshes/head-center.stl" scale="0.001 0.001 0.001"/>
@@ -215,5 +215,5 @@
   <link name="eye_right_link">
     <visual>
-      <origin xyz="0.15 -0.15 -0.15" rpy="0.0 0.0 1.570796327"/> <!--TODO fix origin of mesh-->
+      <origin xyz="0.0 0.0 0.0" rpy="0.0 0.0 0.0"/> <!--TODO fix origin of mesh-->
       <geometry>
         <mesh filename="package://wall_e_description/meshes/eye-right.stl" scale="0.001 0.001 0.001"/>
@@ -229,5 +229,5 @@
   <link name="eye_left_link">
     <visual>
-      <origin xyz="0.15 -0.15 -0.15" rpy="0.0 0.0 1.570796327"/> <!--TODO fix origin of mesh-->
+      <origin xyz="0.0 0.0 0.0" rpy="0.0 0.0 0.0"/> <!--TODO fix origin of mesh-->
       <geometry>
         <mesh filename="package://wall_e_description/meshes/eye-left.stl" scale="0.001 0.001 0.001"/>

Commit message: Update mesh origins and add actual joints to controllable joints of WALL-E

File: ros/wall_e_description/urdf/wall_e.urdf.xacro (robot description, xacro)
@@ -15,5 +15,5 @@
     <parent link="base_footprint"/>
     <child link="base_link"/>
-    <origin xyz="0.0 0.0 0.138887" rpy="0.0 0.0 0.0"/> <!--TODO fix offset of link-->
+    <origin xyz="0.0 0.0 0.138887" rpy="0.0 0.0 0.0"/>
   </joint>
   <link name="base_link">
@@ -82,12 +82,13 @@
     </visual>
   </link>
-  <joint name="wheel_right_joint" type="fixed"> <!--TODO make a continuous joint-->
+  <joint name="wheel_right_joint" type="continuous">
     <parent link="drivetrain_right_link"/>
     <child link="wheel_right_link"/>
-    <origin xyz="0.0 0.0 0.0" rpy="0.0 0.0 0.0"/> <!--TODO fix offset of link-->
+    <origin xyz="-0.049187 -0.1318 -0.103877" rpy="0.0 0.0 0.0"/>
+    <axis xyz="0 1 0"/>
   </joint>
   <link name="wheel_right_link">
     <visual>
-      <origin xyz="0.0 0.0 0.0" rpy="0.0 0.0 0.0"/> <!--TODO fix origin of mesh-->
+      <origin xyz="0.0 0.0 0.0" rpy="0.0 0.0 0.0"/>
       <geometry>
         <mesh filename="package://wall_e_description/meshes/wheel-right.stl" scale="0.001 0.001 0.001"/>
@@ -96,12 +97,13 @@
     </visual>
   </link>
-  <joint name="wheel_left_joint" type="fixed"> <!--TODO make a continuous joint-->
+  <joint name="wheel_left_joint" type="continuous">
     <parent link="drivetrain_left_link"/>
     <child link="wheel_left_link"/>
-    <origin xyz="0.0 0.0 0.0" rpy="0.0 0.0 0.0"/> <!--TODO fix offset of link-->
+    <origin xyz="-0.049187 0.1318 -0.103877" rpy="0.0 0.0 0.0"/>
+    <axis xyz="0 1 0"/>
   </joint>
   <link name="wheel_left_link">
     <visual>
-      <origin xyz="0.0 0.0 0.0" rpy="0.0 0.0 0.0"/> <!--TODO fix origin of mesh-->
+      <origin xyz="0.0 0.0 0.0" rpy="0.0 0.0 0.0"/>
       <geometry>
         <mesh filename="package://wall_e_description/meshes/wheel-left.stl" scale="0.001 0.001 0.001"/>
@@ -110,12 +112,14 @@
     </visual>
   </link>
-  <joint name="arm_right_joint" type="fixed"> <!--TODO make a limited joint-->
+  <joint name="arm_right_joint" type="revolute">
     <parent link="base_link"/>
     <child link="arm_right_link"/>
-    <origin xyz="0.0 0.0 0.0" rpy="0.0 0.0 0.0"/> <!--TODO fix offset of link-->
+    <origin xyz="-0.036105 -0.0725 0.045529" rpy="0.0 0.0 0.0"/>
+    <axis xyz="0 1 0"/>
+    <limit effort="1000.0" lower="-4.0" upper="0.7" velocity="1000.0"/> <!--TODO update for actual limits-->
   </joint>
   <link name="arm_right_link">
     <visual>
-      <origin xyz="0.0 0.0 0.0" rpy="0.0 0.0 0.0"/> <!--TODO fix origin of mesh-->
+      <origin xyz="0.0 0.0 0.0" rpy="0.0 0.0 0.0"/>
       <geometry>
         <mesh filename="package://wall_e_description/meshes/arm-right.stl" scale="0.001 0.001 0.001"/>
@@ -124,12 +128,14 @@
     </visual>
   </link>
-  <joint name="arm_left_joint" type="fixed"> <!--TODO make a limited joint-->
+  <joint name="arm_left_joint" type="revolute">
     <parent link="base_link"/>
     <child link="arm_left_link"/>
-    <origin xyz="0.0 0.0 0.0" rpy="0.0 0.0 0.0"/> <!--TODO fix offset of link-->
+    <origin xyz="-0.036105 0.07275 0.045547" rpy="0.0 0.0 0.0"/>
+    <axis xyz="0 1 0"/>
+    <limit effort="1000.0" lower="-4.0" upper="0.7" velocity="1000.0"/> <!--TODO update for actual limits-->
   </joint>
   <link name="arm_left_link">
     <visual>
-      <origin xyz="0.0 0.0 0.0" rpy="0.0 0.0 0.0"/> <!--TODO fix origin of mesh-->
+      <origin xyz="0.0 0.0 0.0" rpy="0.0 0.0 0.0"/>
       <geometry>
         <mesh filename="package://wall_e_description/meshes/arm-left.stl" scale="0.001 0.001 0.001"/>
@@ -141,9 +147,9 @@
     <parent link="arm_right_link"/>
     <child link="hand_right_link"/>
-    <origin xyz="0.0 0.0 0.0" rpy="0.0 0.0 0.0"/>
+    <origin xyz="0.135 -0.026 0.0" rpy="0.0 0.0 0.0"/>
   </joint>
   <link name="hand_right_link">
     <visual>
-      <origin xyz="0.0 0.0 0.0" rpy="0.0 0.0 0.0"/> <!--TODO fix origin of mesh-->
+      <origin xyz="0.0 0.0 0.0" rpy="0.0 0.0 0.0"/>
       <geometry>
         <mesh filename="package://wall_e_description/meshes/hand-right.stl" scale="0.001 0.001 0.001"/>
@@ -155,9 +161,9 @@
     <parent link="arm_left_link"/>
     <child link="hand_left_link"/>
-    <origin xyz="0.0 0.0 0.0" rpy="0.0 0.0 0.0"/>
+    <origin xyz="0.135 0.041 0.0" rpy="0.0 0.0 0.0"/>
   </joint>
   <link name="hand_left_link">
     <visual>
-      <origin xyz="0.0 0.0 0.0" rpy="0.0 0.0 0.0"/> <!--TODO fix origin of mesh-->
+      <origin xyz="0.0 0.0 0.0" rpy="0.0 0.0 0.0"/>
       <geometry>
         <mesh filename="package://wall_e_description/meshes/hand-left.stl" scale="0.001 0.001 0.001"/>
@@ -166,12 +172,14 @@
     </visual>
   </link>
-  <joint name="neck_bottom_joint" type="fixed"> <!--TODO make a limited joint-->
+  <joint name="neck_bottom_joint" type="revolute">
     <parent link="base_link"/>
     <child link="neck_bottom_link"/>
-    <origin xyz="0.0 0.0 0.0" rpy="0.0 0.0 0.0"/> <!--TODO fix offset of link-->
+    <origin xyz="-0.023342 0.0 0.080" rpy="0.0 0.0 0.0"/>
+    <axis xyz="0 1 0"/>
+    <limit effort="1000.0" lower="-0.5" upper="0.1" velocity="1000.0"/> <!--TODO update for actual limits-->
   </joint>
   <link name="neck_bottom_link">
     <visual>
-      <origin xyz="0.0 0.0 0.0" rpy="0.0 0.0 0.0"/> <!--TODO fix origin of mesh-->
+      <origin xyz="0.0 0.0 0.0" rpy="0.0 0.0 0.0"/>
       <geometry>
         <mesh filename="package://wall_e_description/meshes/neck-bottom.stl" scale="0.001 0.001 0.001"/>
@@ -180,12 +188,14 @@
     </visual>
   </link>
-  <joint name="neck_top_joint" type="fixed"> <!--TODO make a limited joint-->
+  <joint name="neck_top_joint" type="revolute">
     <parent link="neck_bottom_link"/>
     <child link="neck_top_link"/>
-    <origin xyz="0.0 0.0 0.0" rpy="0.0 0.0 0.0"/> <!--TODO fix offset of link-->
+    <origin xyz="0.059852 0.0 0.008848" rpy="0.0 0.0 0.0"/>
+    <axis xyz="0 1 0"/>
+    <limit effort="1000.0" lower="-0.2" upper="1.5" velocity="1000.0"/> <!--TODO update for actual limits-->
   </joint>
   <link name="neck_top_link">
     <visual>
-      <origin xyz="0. 0.0 0.0" rpy="0.0 0.0 0.0"/> <!--TODO fix origin of mesh-->
+      <origin xyz="0. 0.0 0.0" rpy="0.0 0.0 0.0"/>
       <geometry>
         <mesh filename="package://wall_e_description/meshes/neck-top.stl" scale="0.001 0.001 0.001"/>
@@ -194,12 +204,13 @@
     </visual>
   </link>
-  <joint name="head_center_joint" type="fixed"> <!--TODO make a limited joint-->
+  <joint name="head_center_joint" type="continuous"> <!--TODO make a limited joint-->
     <parent link="neck_top_link"/>
     <child link="head_center_link"/>
-    <origin xyz="0.0 0.0 0.0" rpy="0.0 0.0 0.0"/> <!--TODO fix offset of link-->
+    <origin xyz="-0.033445 0.0 0.053725" rpy="0.0 0.0 0.0"/>
+    <axis xyz="0 0 1"/>
   </joint>
   <link name="head_center_link">
     <visual>
-      <origin xyz="0.0 0.0 0.0" rpy="0.0 0.0 0.0"/> <!--TODO fix origin of mesh-->
+      <origin xyz="0.0 0.0 0.0" rpy="0.0 0.0 0.0"/>
       <geometry>
         <mesh filename="package://wall_e_description/meshes/head-center.stl" scale="0.001 0.001 0.001"/>
@@ -208,12 +219,14 @@
     </visual>
   </link>
-  <joint name="eye_right_joint" type="fixed"> <!--TODO make a limited joint-->
+  <joint name="eye_right_joint" type="revolute">
     <parent link="head_center_link"/>
     <child link="eye_right_link"/>
-    <origin xyz="0.0 0.0 0.0" rpy="0.0 0.0 0.0"/> <!--TODO fix offset of link-->
+    <origin xyz="0.075654 0.0 0.028992" rpy="0.0 0.0 0.0"/>
+    <axis xyz="1 0 0"/>
+    <limit effort="1000.0" lower="-0.1" upper="0.3" velocity="1000.0"/> <!--TODO update for actual limits-->
   </joint>
   <link name="eye_right_link">
     <visual>
-      <origin xyz="0.0 0.0 0.0" rpy="0.0 0.0 0.0"/> <!--TODO fix origin of mesh-->
+      <origin xyz="0.0 0.0 0.0" rpy="0.0 0.0 0.0"/>
       <geometry>
         <mesh filename="package://wall_e_description/meshes/eye-right.stl" scale="0.001 0.001 0.001"/>
@@ -222,12 +235,14 @@
     </visual>
   </link>
-  <joint name="eye_left_joint" type="fixed"> <!--TODO make a limited joint-->
+  <joint name="eye_left_joint" type="revolute">
     <parent link="head_center_link"/>
     <child link="eye_left_link"/>
-    <origin xyz="0.0 0.0 0.0" rpy="0.0 0.0 0.0"/> <!--TODO fix offset of link-->
+    <origin xyz="0.075364 0.0 0.0289895" rpy="0.0 0.0 0.0"/>
+    <axis xyz="1 0 0"/>
+    <limit effort="1000.0" lower="-0.3" upper="0.1" velocity="1000.0"/> <!--TODO update for actual limits-->
   </joint>
   <link name="eye_left_link">
     <visual>
-      <origin xyz="0.0 0.0 0.0" rpy="0.0 0.0 0.0"/> <!--TODO fix origin of mesh-->
+      <origin xyz="0.0 0.0 0.0" rpy="0.0 0.0 0.0"/>
       <geometry>
         <mesh filename="package://wall_e_description/meshes/eye-left.stl" scale="0.001 0.001 0.001"/>
